File: Kicad/MicroLit/Microlit.sch (KiCad schematic (older format))
At the start: 23 parts, among them J1 USB_OTG, J10 Conn_01x02, J11 Conn_01x04, J12 Conn_01x03, J13 Conn_01x01, J14 Conn_01x01, J15 Conn_01x01, J16 Conn_01x01, J2 USB_OTG, J3 USB_A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

Commit message: update for v2
Parts:
- C1: value C -> 1uF
- C2: value C -> 10uF
- R1: value R -> 330R
Changed lines of the file:
@@
 LIBS:74LVC1T45Z6-7
 LIBS:Microlit-cache
-EELAYER 27 0
+EELAYER 25 0
 EELAYER END
 $Descr A4 11693 8268
@@
 Sheet 1 1
 Title ""
-Date "3 apr 2019"
+Date ""
 Rev ""
 Comp ""
@@
 P 7000 4750
 F 0 "R1" V 7080 4750 50  0000 C CNN
-F 1 "R" V 7000 4750 50  0000 C CNN
+F 1 "330R" V 7000 4750 50  0000 C CNN
 F 2 "Resistors_SMD:R_0603" V 6930 4750 50  0001 C CNN
 F 3 "" H 7000 4750 50  0001 C CNN
@@
 P 7050 2950
 F 0 "C2" H 7075 3050 50  0000 L CNN
-F 1 "C" H 7075 2850 50  0000 L CNN
+F 1 "10uF" H 7075 2850 50  0000 L CNN
 F 2 "Capacitors_SMD:C_0603" H 7088 2800 50  0001 C CNN
 F 3 "" H 7050 2950 50  0001 C CNN
@@
 P 4700 2950
 F 0 "C1" H 4725 3050 50  0000 L CNN
-F 1 "C" H 4725 2850 50  0000 L CNN
+F 1 "1uF" H 4725 2850 50  0000 L CNN
 F 2 "Capacitors_SMD:C_0603" H 4738 2800 50  0001 C CNN
 F 3 "" H 4700 2950 50  0001 C CNN
